File: PSU.sch (EAGLE design)
At the start: 40 parts, among them IC1 7812T, IC2 LM7912, Q1 TIP120, Q2 TIP125, X1 332-16, X10 332-16, X11 332-16, X12 332-16, X13 332-16, X14 332-16, X2 332-16, X3 332-16, X4 332-16, X5 332-16, X6 332-16, X7 332-16, X8 332-16, X9 332-16

Commit message: A different approach
Parts:
- added C11: 2.2nF, rcl:C-EUC0805
- added C12: 6.8uF, rcl:C-EUC0805
- added C13, C14: 4.7uF, rcl:C-EUC0805
- added C15: 100uF, rcl:CPOL-EUE7.5-16
- added C16, C17: 10uF, rcl:CPOL-EUB
- added C18: 2200uF, rcl:CPOL-EUE7.5-16
- added C19: 1uF, rcl:CPOL-EUE7.5-16
- added C20: 2.2uF, rcl:CPOL-EUE7.5-16
- added D3, D4: 1N4004, diode:1N4004
- added IC3: LM7912, v-reg:79XXL
- added L1XAL4020-102MEB: 1uH, rcl:L-EUL5038P
- added Q3: TIP125, transistor-power:TIP125
- added R6: 1.62M, rcl:R-EU_R0805
- added R7, R8: 100k, rcl:R-EU_R0805
- added R9: 1k, rcl:R-EU_R0805
- added U2: Value, texas12vsupply:TPS62135RGXR
Connections:
- removed net +24V: C10.+, C2.+, C3.1, C6.+, CN1.PWR, IC1.VI, U$1.TIP
- removed net GNDA: C1.-, C4.2, C5.-, C9.-, CN1.GND, CN1.GNDBREAK, IC2.IN, U$1.RING, U$1.RING_SW
- new net +15V: C12.1, CN1.PWR, U$1.TIP, U2.VIN
- new net 10: U2.EN
- new net 14P4: C17.+, L1XAL4020-102MEB.1, U2.SW
- new net N$1: R8.2, U2.PG
- new net N$10: C11.1, U2.SS_TR
- new net N$11: R6.1, R7.2, U2.FB
- new net N$12: C16.-, Q3.B, R9.1
- new net N$13: C17.-, D3.A, D4.C
- new net N$3: C15.-, C18.-, C20.-, D4.A, IC3.IN
- new net N$7: C10.+, C2.+, C3.1, C6.+, IC1.VI
- new net N$8: C1.-, C4.2, C5.-, C9.-, IC2.IN
- new net N$9: C19.-, IC3.OUT, Q3.C, R9.2
- net +12V: now also C13.1, C14.1, L1XAL4020-102MEB.2, R6.2, R8.1, U2.VOS
- net -12V: now also Q3.E
- net GND: now also C11.2, C12.2, C13.2, C14.2, C15.+, C16.+, C18.+, C19.+, C20.+, CN1.GND, CN1.GNDBREAK, D3.C, IC3.GND, R7.1, U$1.RING, U$1.RING_SW, U2.FB2, U2.GND, U2.MODE, U2.VSEL
Other:
- moved on the sheet: C1, C10, C2, C3, C4, C5, C6, C7, C8, C9, CN1, D1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

Commit message: Update
Parts:
- removed C1, C10, C18, C2, C5, C6, C9: 2200uF, rcl:CPOL-EUE7.5-16
- removed C3, C4: 22uF, rcl:C-EU025-025X050
- removed C7, C8: 10uF, rcl:C-EU025-025X050
- removed D1, D2: 1N4004, diode:1N4004
- removed IC1: 7812T, linear:7812T
- removed IC2: LM7912, v-reg:79XXL
- removed Q1: TIP120, transistor-power:TIP120
- removed Q2, Q3: TIP125, transistor-power:TIP125
- removed R1, R2: 1k, rcl:R-EU_0207/7
- removed X10, X11, X12, X13, X14, X9: 332-16, con-garry:332-16
- added U$2: MPS751, audioic:MPS751
- C15, C19, C20: device rcl:CPOL-EUE7.5-16 -> rcl:CPOL-EUB
- C16: value 10uF -> 100uF
Connections:
- removed net N$2: IC2.OUT, Q2.E, R2.1
- removed net N$4: IC1.VO, Q1.C, R1.1
- removed net N$5: C7.1, Q1.B, R1.2
- removed net N$6: C8.2, Q2.B, R2.2
- removed net N$7: C10.+, C2.+, C3.1, C6.+, IC1.VI
- removed net N$8: C1.-, C4.2, C5.-, C9.-, IC2.IN
- net +12V: no longer D1.C, Q1.E, X10-10.S, X10-9.S, X11-10.S, X11-9.S, X12-10.S, X12-9.S, X13-10.S, X13-9.S, X14-10.S, X14-9.S, X9-10.S, X9-9.S
- net +5V: no longer X10-11.S, X10-12.S, X11-11.S, X11-12.S, X12-11.S, X12-12.S, X13-11.S, X13-12.S, X14-11.S, X14-12.S, X9-11.S, X9-12.S
- net -12V: now also U$2.E; no longer D2.A, Q2.C, Q3.E, X10-1.S, X10-2.S, X11-1.S, X11-2.S, X12-1.S, X12-2.S, X13-1.S, X13-2.S, X14-1.S, X14-2.S, X9-1.S, X9-2.S
- net GND: no longer C1.+, C10.-, C18.+, C2.-, C3.2, C4.1, C5.+, C6.-, C7.2, C8.1, C9.+, D1.A, D2.C, IC1.GND, IC2.GND, X10-3.S, X10-4.S, X10-5.S, X10-6.S, X10-7.S, X10-8.S, X11-3.S, X11-4.S, X11-5.S, X11-6.S, X11-7.S, X11-8.S, X12-3.S, X12-4.S, X12-5.S, X12-6.S, X12-7.S, X12-8.S, X13-3.S, X13-4.S, X13-5.S, X13-6.S, X13-7.S, X13-8.S, X14-3.S, X14-4.S, X14-5.S, X14-6.S, X14-7.S, X14-8.S, X9-3.S, X9-4.S, X9-5.S, X9-6.S, X9-7.S, X9-8.S
- net N$12: now also U$2.B; no longer Q3.B
- net N$19: no longer X10-15.S, X10-16.S, X11-15.S, X11-16.S, X12-15.S, X12-16.S, X13-15.S, X13-16.S, X14-15.S, X14-16.S, X9-15.S, X9-16.S
- net N$20: no longer X10-13.S, X10-14.S, X11-13.S, X11-14.S, X12-13.S, X12-14.S, X13-13.S, X13-14.S, X14-13.S, X14-14.S, X9-13.S, X9-14.S
- net N$3: no longer C18.-
- net N$9: now also U$2.C; no longer Q3.C
Other:
- moved on the sheet: C16, R9
